File: PushItDIP/schematic/Push-It-V1.0.sch (EAGLE design)
At the start: 30 parts, among them IC1 74LS595N, IC2 ATMEGA328P-PU, Q1 16MHZ

Commit message: PushItDIP: Changed Resistor R6 from 33k to 1k
Parts:
- R6: value 33k -> 1k
