File: PushItDIP/schematic/Push-It-V1.1.brd (EAGLE design)
At the start: 63.5 x 84.8 mm, 30 parts, among them IC1 74LS595N, IC2 ATMEGA328P-PU, Q1 16MHZ

Commit message: PushItDIP: Finished documentation and adjusted resistor value
Parts:
- R6: value 1k -> 220
Changed lines of the file:
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@@
 <attribute name="VALUE" x="31.1912" y="40.386" size="1.27" layer="27" ratio="10" rot="R270"/>
 </element>
-<element name="R6" library="rcl" package="0207/7" value="1k" x="31.75" y="63.5" smashed="yes" rot="R270">
+<element name="R6" library="rcl" package="0207/7" value="220" x="31.75" y="63.5" smashed="yes" rot="R270">
 <attribute name="NAME" x="33.147" y="66.04" size="1.27" layer="25" ratio="10" rot="R270"/>
 <attribute name="VALUE" x="31.1912" y="65.786" size="1.27" layer="27" ratio="10" rot="R270"/>
